File: kicad_v1/firefly/firefly.kicad_sch (KiCad schematic)
At the start: 18 parts, among them J1 SEL_CA_CC, J2 ISP, J3 Vin, J4 Vout, Q1 SHF3310, U1 ATtiny13A-P

Commit message: added code
Parts:
- added J5, J6: Vout, firefly:PinHeader_1x02_P2.54mm_Vertical, symbol firefly:Conn_01x02
- J4: value Vout -> Vin
Connections:
- net GND: now also J5.2 (Pin_2), J6.2 (Pin_2)
- net VCC: now also J5.1 (Pin_1), J6.1 (Pin_1)
Other:
- moved on the sheet: J3, J4
